File: hardware/orangecrab_r0.2.1/IO.kicad_sch (KiCad schematic)
At the start: 37 parts, among them J3 USB_C_Receptacle_USB2.0, SW1 SW_Push, U9 74HC4067BQ

Commit message: kicad9 update
Parts:
- gave numbers to parts that had none: 2
