File: hardware/orangecrab_r0.2.1/OrangeCrab.kicad_pcb (KiCad board)
At the start: 6 copper layers, 50.8 x 22.9 mm, 163 parts, among them J1 Conn_01x12_Male, J2 Conn_01x16_Male, J3 USB_C_Receptacle_USB2.0, J4 MicroSd, J5 JST, J6 Conn_01x05_Male, SW1 SW_Push, U1 TLV62569DRL, U10 NCP115-2.5, U2 TLV62569DRL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

Commit message: kicad7 update
Other:
- net class DDR3_CTRL_LM1.0 removed
- net class DDR3_DQS0_LM1.0 removed
- net class DDR3_DQS1_LM1.0 removed
- net class DDR_CLK_LM1.0 removed
- net class Default removed
